File: hackboard.sch (KiCad schematic (older format))
At the start: 81 parts, among them J1 USB, P1 CONN_4, P10 CONN_2, P11 CONN_2, P12 CONN_2, P13 CONN_2, P14 CONN_2, P15 CONN_2, P16 CONN_2X2, P2 CONN_4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

Commit message: Change IR2184 to Vdd instead of Vcc
Parts:
- added C32: C, symbol C
- added P17: CONN_2, symbol CONN_2
- C14: value 10nF -> 4.7uF
- C15: value 10nF -> 100nF
- C16, C17, C19: value 10nF -> 100nf
- R34: value 1M1 -> 1M
Connections:
- wire segments 297 -> 301

Commit message: Added second power connector
Parts:
- removed J1: USB, symbol USB
- added D15: LED, symbol LED
- added P18: CONN_1, symbol CONN_1
- added R35: 1k, symbol R
- added U12: MICRO-B_USB, symbol MICRO-B_USB
Connections:
- wire segments 301 -> 296
- no-connect marks 15 -> 16

Commit message: Recovered from hdd!
Parts:
- added P19: CONN_2, symbol CONN_2

Commit message: fixed gnd/vcc flips
Parts:
- removed U12: MICRO-B_USB, symbol MICRO-B_USB
- removed U4: STM32L100XX_LQFP64, MODULE, symbol STM32L100XX_LQFP64
- added CON?: USB-MINI-B, symbol USB-MINI-B
- added U?: STM32L100xx_LQFP64, MODULE, symbol STM32L100xx_LQFP64
- X1: value 20MHz -> 8MHz
Connections:
- wire segments 296 -> 353
- no-connect marks 16 -> 15

Commit message: didn't save everyting
Parts:
- gave numbers to parts that had none: 2
